File: Teensy4.1-example.kicad_sch (KiCad schematic)
At the start: 80 parts, among them IC1 MIMXRT1062DVJ6B, J1 Conn_01x11_Male, J2 Conn_01x11_Male, J3 Conn_01x12_Male, J4 Conn_01x11_Male, J5 Conn_01x11_Male, J6 Conn_01x03_Male, J7 Conn_01x03_Male, P2 D26, Q1 Q_PMOS_GDS_DMP3125L, U1 opto_APA102-2020, U2 MAX1562, U3 W25Q64JVXGIM, U4 MKL02Z32VFG4, Y1 Crystal_GND23, Y2 Crystal

Commit message: Modified
Parts:
- removed D2: LED, LED_SMD:LED_0402_1005Metric, symbol Device:LED
- removed Di3: SP0503BAHT, Package_TO_SOT_SMD:SOT-143, symbol Power_Protection:SP0503BAHT
- removed J1, J2, J4, J5: Conn_01x11_Male, Connector_PinHeader_2.54mm:PinHeader_1x11_P2.54mm_Vertical, symbol Connector:Conn_01x11_Male
- removed J3: Conn_01x12_Male, Connector_PinHeader_2.54mm:PinHeader_1x12_P2.54mm_Vertical, symbol Connector:Conn_01x12_Male
- removed J6: Conn_01x03_Male, Connector_PinHeader_2.54mm:PinHeader_1x03_P2.54mm_Vertical, symbol Connector:Conn_01x03_Male
- removed P2: D26, Connector_PinHeader_1.00mm:PinHeader_1x01_P1.00mm_Vertical, symbol Connector:TestPoint
- removed R12, R13: 56k, Resistor_SMD:R_0603_1608Metric, symbol Device:R
- removed R16: 100k, Resistor_SMD:R_0603_1608Metric, symbol Device:R
- removed R6, R7: 16k, Resistor_SMD:R_0603_1608Metric, symbol Device:R
- removed R8: 1k, Resistor_SMD:R_0402_1005Metric, symbol Device:R
- removed R9: 1M, Resistor_SMD:R_0603_1608Metric, symbol Device:R
- removed U1: opto_APA102-2020, USB-C-Power-tester:APA102-2020, symbol APA102:opto_APA102-2020
- removed U2: MAX1562, Package_SO:SO-8_3.9x4.9mm_P1.27mm, symbol MIMXRT1062DVJ6B:MAX1562
- removed USB_DFP1: USB_C_Receptacle_USB2.0, USB-C-Power-tester:TYPE-C-31-M-14, symbol simonsen:USB_C_Receptacle_USB2.0_NOPOW
- added H1, H2, H3: MountingHole, MountingHole:MountingHole_2.7mm_M2.5_DIN965_Pad_TopBottom, symbol Mechanical:MountingHole
- added H4: MountingHole, MountingHole:MountingHole_2.7mm_M2.5_DIN965_Pad_TopBottom, symbol Mechanical:MountingHole_Pad
- added J1, J2: Conn_01x20, Connector_FFC-FPC:Hirose_FH12-20S-0.5SH_1x20-1MP_P0.50mm_Horizontal, symbol Connector_Generic:Conn_01x20
- USB_UFP1: footprint USB-C-Power-tester:TYPE-C-31-M-14 -> acheron_Connectors:USB_C_Receptacle_Hroparts_TYPE-C-31-M-12
- renumbered C18 to C13, C19 to C14, C20 to C15, C21 to C16, C13 to C17, C14 to C18, C15 to C19, C16 to C20, C22 to C21, C17 to C22, D3 to D2, D5 to D3, J7 to J3, NCP692 to NCP1, R14 to R6, R15 to R7, R10 to R8, R11 to R9, U3 to U1, U4 to U2
Connections:
- net +3V3: now also J1.1 (Pin_1)
- net +5V: now also J1.2 (Pin_2)
- net GND: now also H4.1, J2.19 (Pin_19), J2.20 (Pin_20)
- net R1: now reaches IC1.B1 (GPIO_EMC_15)
- net R1: now also J1.3 (Pin_3)
- net D0 renamed L0
- net L0: now also J2.1 (Pin_1)
- net D1 renamed L1
- net L1: now also J2.2 (Pin_2)
- net D10: no longer names the net of IC1.D7 (GPIO_B0_00)
- net D11: no longer names the net of IC1.E8 (GPIO_B0_02)
- net D12: no longer names the net of IC1.E7 (GPIO_B0_01)
- net D14_A0 renamed L2
- net L2: now also J2.3 (Pin_3)
- net D15_A1 renamed L3
- net L3: now also J2.4 (Pin_4)
- net D16_A2 renamed L14
- net L14: now also J2.15 (Pin_15)
- net D17_A3 renamed L12
- net L12: now also J2.13 (Pin_13)
- net D18_A4: no longer names the net of IC1.K11 (GPIO_AD_B1_01)
- net D19_A5 renamed L13
- net L13: now also J2.14 (Pin_14)
- net D2 renamed R10
- net R10: now also J1.12 (Pin_12)
- net D20_A6 renamed L5
- net L5: now also J2.6 (Pin_6)
- net D21_A7 renamed L16
- net L16: now also J2.17 (Pin_17)
- net D22_A8 renamed L10
- net L10: now also J2.11 (Pin_11)
- net D23_A9 renamed L4
- net L4: now also J2.5 (Pin_5)
- net D24_A10 renamed L7
- net L7: now also J2.8 (Pin_8)
- net D25_A11 renamed L6
- net L6: now also J2.7 (Pin_7)
- net D26_A12 renamed L11
- net L11: now also J2.12 (Pin_12)
- net D27_A13 renamed L15
- net L15: now also J2.16 (Pin_16)
- net D28: no longer names the net of IC1.D5 (GPIO_EMC_32)
- net D29: no longer names the net of IC1.C5 (GPIO_EMC_31)
- net D3 renamed R9
- net R9: now also J1.11 (Pin_11)
- net D30 renamed R6
- net R6: now also J1.8 (Pin_8)
- net D31 renamed R2
- net R2: now also J1.4 (Pin_4)
- net D32: no longer names the net of IC1.C10 (GPIO_B0_12)
- net D33 renamed R12
- net R12: now also J1.14 (Pin_14)
- net D34: no longer names the net of IC1.D14 (GPIO_B1_13)
- net D35: no longer names the net of IC1.D13 (GPIO_B1_12)
- net D36: no longer names the net of IC1.C11 (GPIO_B1_02)
- net D37: no longer names the net of IC1.D11 (GPIO_B1_03)
- net D38_A14 renamed L9
- net L9: now also J2.10 (Pin_10)
- net D39_A15 renamed L8
- net L8: now also J2.9 (Pin_9)
- net D4 renamed R14
- net R14: now also J1.16 (Pin_16)
- net D40_A16 renamed L17
- net L17: now also J2.18 (Pin_18)
- net D41_A17: no longer names the net of IC1.K12 (GPIO_AD_B1_05)
- net D42 renamed R18
- net R18: now also J1.20 (Pin_20)
- net D43 renamed R15
- net R15: now also J1.17 (Pin_17)
- net D44 renamed R13
- net R13: now also J1.15 (Pin_15)
- net D45 renamed R17
- net R17: now also J1.19 (Pin_19)
- net D46 renamed R16
- net R16: now also J1.18 (Pin_18)
- net D48 renamed R3
- net R3: now also J1.5 (Pin_5)
- net D49: no longer names the net of IC1.A2 (GPIO_EMC_27)
- net D5 renamed R11
- net R11: now also J1.13 (Pin_13)
- net D50 renamed R5
- net R5: now also J1.7 (Pin_7)
- net D51 renamed R8
- net R8: now also J1.10 (Pin_10)
- net D52: no longer names the net of IC1.B3 (GPIO_EMC_26)
- net D53 renamed R4
- net R4: now also J1.6 (Pin_6)
- net D54 renamed R7
- net R7: now also J1.9 (Pin_9)
- net D6: no longer names the net of IC1.D9 (GPIO_B0_10)
- net D7: no longer names the net of IC1.B11 (GPIO_B1_01)
- net D8: no longer names the net of IC1.A11 (GPIO_B1_00)
- net D9: no longer names the net of IC1.A10 (GPIO_B0_11)
- net USB2_DN: no longer names the net of IC1.N7 (USB_OTG2_DN)
- net USB2_DP: no longer names the net of IC1.P7 (USB_OTG2_DP)
- no-connect marks 66 -> 82
